Commit message: rising_description: current wheel definition

File: rising_description/urdf/wheels/wheel.gazebo.xacro (robot description, xacro)
@@ -2,16 +2,15 @@
 <robot xmlns:xacro="http://www.ros.org/wiki/xacro">
     <xacro:macro name="wheel_gazebo" params="prefix">
-        <gazebo reference="${prefix}_wheel_link">
-            <mu1 value="10000"/>
-			      <mu2 value="10000"/>
-			      <kp value="10000000.0" />
+        <gazebo reference="${prefix}link">
+            <mu1 value="100.0"/>
+			      <mu2 value="100.0"/>
+ 			      <kp value="10000000.0" />
 			      <kd value="1.0" />
 		      	<fdir1 value="1 0 0"/>
-			<material>Gazebo/Yellow</material>
-            <turnGravityOff>false</turnGravityOff>
+			      <material>Gazebo/Yellow</material>
         </gazebo>
     </xacro:macro>
     <!-- Gazebo Mimic Joints Plugin -->
-  <xacro:macro name="mimic_joint_plugin_gazebo" params="prefix parent_joint mimic_joint has_pid:=false multiplier:=1 offset:=0 sensitiveness:=0.0 max_effort:=1.0 robot_namespace:=''">
+  <xacro:macro name="mimic_joint_plugin_gazebo" params="prefix parent_joint mimic_joint has_pid:=false multiplier offset:=0 sensitiveness:=0.0 max_effort:=1.0 robot_namespace:=''">
     <gazebo>
       <plugin name="${prefix}mimic_joint_plugin" filename="libroboticsgroup_gazebo_mimic_joint_plugin.so">

File: rising_description/urdf/wheels/wheel.transmission.xacro (robot description, xacro)
@@ -4,10 +4,10 @@
     <xacro:macro name="wheel_transmission" params="prefix">
     <!-- Transmission is important to link the joints and the controller (see rising_control/config/rising_control.yaml)-->
-        <transmission name="${prefix}master_wheel_joint_trans" params="prefix">
+        <transmission name="${prefix}joint_trans" params="prefix">
             <type>transmission_interface/SimpleTransmission</type>
-            <joint name="${prefix}master_wheel_joint">
+            <joint name="${prefix}joint">
                 <hardwareInterface>hardware_interface/VelocityJointInterface</hardwareInterface>
             </joint>
-            <actuator name="${prefix}master_wheel_joint_motor">
+            <actuator name="${prefix}joint_motor">
 				<mechanicalReduction>1</mechanicalReduction>
 				<motorTorqueConstant>20</motorTorqueConstant>

File: rising_description/urdf/wheels/wheel.urdf.xacro (robot description, xacro)
@@ -8,12 +8,12 @@
 	<xacro:property name="master_wheel_radius" value="0.09256"/>
 	<xacro:property name="master_wheel_width" value="0.047"/>
-  <xacro:property name="master_wheel_mass" value="1"/><!-- in kg-->
+  <xacro:property name="master_wheel_mass" value="5"/><!-- in kg-->
   <xacro:property name="slave_wheel2345_radius" value="0.04148"/>
 	<xacro:property name="slave_wheel2345_height" value="0.047"/>
-  <xacro:property name="slave_wheel2345_mass" value="0.5"/> <!-- in kg-->
-  <xacro:property name="slave_wheel6_radius" value="0.053205"/>
-	<xacro:property name="slave_wheel6_height" value="0.047"/>
-  <xacro:property name="slave_wheel6_mass" value="0.1"/> <!-- in kg-->
- 	<xacro:property name="multiplier_mid_wheel" value="${master_wheel_radius/slave_wheel6_radius}"/>
+  <xacro:property name="slave_wheel2345_mass" value="5"/> <!-- in kg-->
+  <xacro:property name="mid_wheel_radius" value="0.053205"/>
+	<xacro:property name="mid_wheel_width" value="0.047"/>
+  <xacro:property name="mid_wheel_mass" value="5"/> <!-- in kg-->
+ 	<xacro:property name="multiplier_mid_wheel" value="${master_wheel_radius/mid_wheel_radius}"/>
   <xacro:property name="multiplier_small_wheel" value="${master_wheel_radius/slave_wheel2345_radius}"/>
   <xacro:macro name="wheel" params="prefix parent y_origin reflect">
@@ -23,5 +23,5 @@
       <origin xyz="0 ${y_origin} 0" rpy="0 0 0"/>
       <axis xyz="0 1 0" rpy="0 0 0"/>
-      <limit effort="100" velocity="100"/>
+      <limit effort="10" velocity="10"/>
       <joint_properties damping="0.0" friction="0.0"/>
     </joint>
@@ -54,5 +54,5 @@
     <joint name="${prefix}small_wheel_joint" type="continuous">
       <parent link="${parent}"/>
-      <child link="${prefix}slave_wheel_link"/>
+      <child link="${prefix}small_wheel_link"/>
       <xacro:if value="${reflect}">
         <origin xyz="0.08227 ${y_origin} -0.08227" rpy="0 0 0"/>
@@ -62,10 +62,10 @@
       </xacro:unless>
       <axis xyz="0 1 0" rpy="0 0 0"/>
-      <limit effort="100" velocity="100"/>
+      <limit effort="10" velocity="10"/>
       <mimic joint="{prefix}master_wheel_joint" multiplier="${multiplier_small_wheel}" offset="0" />
       <joint_properties damping="0.0" friction="0.0"/>
     </joint>
     <!-- R2: Second link is the down-inside pulley -->
-    <link name="${prefix}slave_wheel_link">
+    <link name="${prefix}small_wheel_link">
       <visual>
         <origin xyz="0 0 0" rpy="0 0 0"/>
@@ -102,5 +102,5 @@
       </xacro:unless>
       <axis xyz="0 1 0" rpy="0 0 0"/>
-      <limit effort="100" velocity="100"/>
+      <limit effort="10" velocity="10"/>
       <mimic joint="{prefix}master_wheel_joint" multiplier="${multiplier_small_wheel}" offset="0" />
       <joint_properties damping="0.0" friction="0.0"/>
@@ -142,5 +142,5 @@
       </xacro:unless>
       <axis xyz="0 1 0" rpy="0 0 0"/>
-      <limit effort="100" velocity="100"/>
+      <limit effort="10" velocity="10"/>
       <mimic joint="{prefix}master_wheel_joint" multiplier="${multiplier_small_wheel}" offset="0" />
       <joint_properties damping="0.0" friction="0.0"/>
@@ -182,5 +182,5 @@
       </xacro:unless>
       <axis xyz="0 1 0" rpy="0 0 0"/>
-      <limit effort="100" velocity="100"/>
+      <limit effort="10" velocity="10"/>
       <mimic joint="{prefix}master_wheel_joint" multiplier="${multiplier_small_wheel}" offset="0" />
       <joint_properties damping="0.0" friction="0.0"/>
@@ -212,7 +212,7 @@
       </inertial>
     </link>
-    <joint name="${prefix}small_wheel_4_joint" type="continuous">
-      <parent link="${parent}"/>
-      <child link="${prefix}small_wheel_4_link"/>
+    <joint name="${prefix}mid_wheel_joint" type="continuous">
+      <parent link="${parent}"/>
+      <child link="${prefix}mid_wheel_link"/>
       <xacro:if value="${reflect}">
         <origin xyz="-0.23515 ${y_origin} 0.03979" rpy="0 0 0"/>
@@ -222,10 +222,10 @@
       </xacro:unless>
       <axis xyz="0 1 0" rpy="0 0 0"/>
-      <limit effort="100" velocity="100"/>
+      <limit effort="10" velocity="10"/>
       <mimic joint="{prefix}master_wheel_joint" multiplier="${multiplier_mid_wheel}" offset="0" />
       <joint_properties damping="0.0" friction="0.0"/>
     </joint>
     <!-- R6: Sixth link is the front pulley -->
-    <link name="${prefix}small_wheel_4_link">
+    <link name="${prefix}mid_wheel_link">
       <visual>
         <origin xyz="0 0 0" rpy="0 0 0"/>
@@ -247,16 +247,16 @@
       </collision-->
       <inertial>
-        <mass value="${slave_wheel6_mass}"/>
-        <origin xyz="0 0 0" rpy="${M_PI/2} 0 0"/>
-        <solid_cylinder_inertia  m="${slave_wheel6_mass}" r="${slave_wheel6_radius}" h="${slave_wheel6_height}"/>
-      </inertial>
-    </link>
-    <xacro:wheel_transmission prefix="${prefix}"/>
-    <xacro:wheel_gazebo prefix="${prefix}"/>
+        <mass value="${mid_wheel_mass}"/>
+        <origin xyz="0 0 0" rpy="${M_PI/2} 0 0"/>
+        <solid_cylinder_inertia  m="${mid_wheel_mass}" r="${mid_wheel_radius}" h="${mid_wheel_width}"/>
+      </inertial>
+    </link>
+    <xacro:wheel_transmission prefix="${prefix}master_wheel_"/>
+    <xacro:wheel_gazebo prefix="${prefix}master_wheel_"/>
+    <xacro:mimic_joint_plugin_gazebo prefix="${prefix}" parent_joint="${prefix}master_wheel_joint" mimic_joint="${prefix}small_wheel_joint" multiplier="${multiplier_small_wheel}"/>
     <xacro:mimic_joint_plugin_gazebo prefix="${prefix}" parent_joint="${prefix}master_wheel_joint" mimic_joint="${prefix}small_wheel_1_joint" multiplier="${multiplier_small_wheel}"/>
     <xacro:mimic_joint_plugin_gazebo prefix="${prefix}" parent_joint="${prefix}master_wheel_joint" mimic_joint="${prefix}small_wheel_2_joint" multiplier="${multiplier_small_wheel}"/>
     <xacro:mimic_joint_plugin_gazebo prefix="${prefix}" parent_joint="${prefix}master_wheel_joint" mimic_joint="${prefix}small_wheel_3_joint" multiplier="${multiplier_small_wheel}"/>
-    <xacro:mimic_joint_plugin_gazebo prefix="${prefix}" parent_joint="${prefix}master_wheel_joint" mimic_joint="${prefix}small_wheel_4_joint" multiplier="${multiplier_mid_wheel}"/>
-    <xacro:mimic_joint_plugin_gazebo prefix="${prefix}" parent_joint="${prefix}master_wheel_joint" mimic_joint="${prefix}small_wheel_joint" multiplier="${multiplier_small_wheel}"/>
-    </xacro:macro>
+    <xacro:mimic_joint_plugin_gazebo prefix="${prefix}" parent_joint="${prefix}master_wheel_joint" mimic_joint="${prefix}mid_wheel_joint" multiplier="${multiplier_mid_wheel}"/>
+  </xacro:macro>
 </robot>
