Commit message: rising_description: solve wrong flippers' collision and add pulleys to simulate the tracked wheels

File: rising_description/urdf/flippers/back_flipper.urdf.xacro (robot description, xacro)
@@ -14,5 +14,5 @@
 	<xacro:property name="lenght_on_z" value="0.196"/>
 	<xacro:property name="y_origin" value="0.274"/>
-    <xacro:macro name="back_flipper" params="prefix parent *origin hq">
+    <xacro:macro name="back_flipper" params="prefix parent *origin">
         <joint name="${prefix}flipper_joint" type="continuous">
             <parent link="${parent}"/>
@@ -25,38 +25,15 @@
         <link name="${prefix}flipper_link">
             <visual>
-                <xacro:if value="${hq}">
-                    <origin xyz="0 0 0" rpy="0 0 0"/>
-                    <geometry>
-                        <mesh filename="package://rising_description/meshes/flippers/back_flippers_final.dae"/>
-                    </geometry>
-                </xacro:if>
-                <xacro:unless value="${hq}">
-                    <origin xyz="0 0 0" rpy="0 0 0"/>
-                    <!-- change geometry if hq!=true -->
-                    <geometry>
-                        <cylinder length="${back_flipper_height}" radius="${back_flipper_radius}"/>
-                    </geometry>
-                </xacro:unless>
+                <origin xyz="0 0 0" rpy="0 0 0"/>
+                <geometry>
+                    <mesh filename="package://rising_description/meshes/flippers/back_flipper.stl"/>
+                </geometry>
             </visual>
-            <collision>
-                  <xacro:if value="${hq}">
-                    <origin xyz="-0.13688 0 0" rpy="${M_PI/2} 0 0"/>
-                    <geometry>
-                        <mesh filename="package://rising_description/meshes/flippers/collision_back_flippers_final.dae" scale="0.001 0.001 0.001"/>
-                    </geometry>
-                </xacro:if>
-                <xacro:unless value="${hq}">
-                    <origin xyz="-0.13688 0 0" rpy="${M_PI/2} 0 0"/>
-                    <!-- change geometry if hq!=true -->
-                    <geometry>
-                        <cylinder length="${back_flipper_height}" radius="${back_flipper_radius}"/>
-                    </geometry>
-                </xacro:unless>
-              <!--origin xyz="0 0 0" rpy="0 0 0"/>
-               <geometry>
-                   <mesh filename="package://rising_description/meshes/flippers/collision_back_flippers.dae" />
-                   <!- - <cylinder length="${back_flipper_height}" radius="${back_flipper_radius}" /> - ->
-               </geometry-->
-            </collision>
+            <!--collision>
+                <origin xyz="0 0 0" rpy="0 0 0"/>
+                <geometry>
+                    <mesh filename="package://rising_description/meshes/flippers/back_flipper.stl"/>
+                </geometry>
+            </collision-->
             <inertial>
                 <mass value="${back_flipper_mass}"/>
@@ -65,6 +42,6 @@
             </inertial>
         </link>
-        <xacro:wheel prefix="${prefix}left_" parent="${prefix}flipper_link" y_origin="${y_origin}" reflect="true" hq="${hq}"/>
-        <xacro:wheel prefix="${prefix}right_" parent="${prefix}flipper_link" y_origin="-${y_origin}" reflect="true" hq="${hq}"/>
+        <xacro:wheel prefix="${prefix}left_" parent="${prefix}flipper_link" y_origin="${y_origin}" reflect="true"/>
+        <xacro:wheel prefix="${prefix}right_" parent="${prefix}flipper_link" y_origin="-${y_origin}" reflect="true"/>
         <xacro:flipper_transmission prefix="${prefix}"/>
         <xacro:back_flipper_gazebo prefix="${prefix}"/>

File: rising_description/urdf/flippers/front_flipper.urdf.xacro (robot description, xacro)
@@ -13,6 +13,6 @@
 	<xacro:property name="lenght_on_y" value="0.65"/>
 	<xacro:property name="lenght_on_z" value="0.196"/>
-	<xacro:property name="y_origin" value="0.274"/>
-    <xacro:macro name="front_flipper" params="prefix parent *origin hq">
+	<xacro:property name="y_origin" value="0.278"/>
+    <xacro:macro name="front_flipper" params="prefix parent *origin">
         <joint name="${prefix}flipper_joint" type="continuous">
             <parent link="${parent}"/>
@@ -25,38 +25,15 @@
         <link name="${prefix}flipper_link">
             <visual>
-                <xacro:if value="${hq}">
-                    <origin xyz="0 0 0" rpy="0 0 0"/>
-                    <geometry>
-                        <mesh filename="package://rising_description/meshes/flippers/front_flippers_final.dae"/>
-                    </geometry>
-                </xacro:if>
-                <xacro:unless value="${hq}">
-                    <origin xyz="0 0 0" rpy="0 0 0"/>
-                    <!-- change geometry if hq!=true -->
-                    <geometry>
-                        <cylinder length="${front_flipper_height}" radius="${front_flipper_radius}"/>
-                    </geometry>
-                </xacro:unless>
+                <origin xyz="0 0 0" rpy="0 0 0"/>
+                <geometry>
+                    <mesh filename="package://rising_description/meshes/flippers/front_flipper.stl"/>
+                </geometry>
             </visual>
-            <collision>
-              <xacro:if value="${hq}">
-                    <origin xyz="0 0 0" rpy="0 0 0"/>
-                    <geometry>
-                        <mesh filename="package://rising_description/meshes/flippers/collision_front_flippers_final.dae" scale="0.001 0.001 0.001"/>
-                    </geometry>
-                </xacro:if>
-                <xacro:unless value="${hq}">
-                    <origin xyz="0 0 0" rpy="0 0 0"/>
-                    <!-- change geometry if hq!=true -->
-                    <geometry>
-                        <cylinder length="${front_flipper_height}" radius="${front_flipper_radius}"/>
-                    </geometry>
-                </xacro:unless>
-                <!-- origin xyz="0 0 0" rpy="0 0 0"/>
+            <!--collision>
+                <origin xyz="0 0 0" rpy="0 0 0"/>
                 <geometry>
-                   <mesh filename="package://rising_description/meshes/flippers/collision_front_flippers.dae" />
-                    <!- - <cylinder length="${front_flipper_height}" radius="${front_flipper_radius}" />- ->
-                </geometry-->
-            </collision>
+                    <mesh filename="package://rising_description/meshes/flippers/front_flipper.stl"/>
+                </geometry>
+            </collision-->
             <inertial>
                 <mass value="${front_flipper_mass}"/>
@@ -65,6 +42,6 @@
             </inertial>
         </link>
-        <xacro:wheel prefix="${prefix}left_" parent="${prefix}flipper_link" y_origin="${y_origin}" reflect="false" hq="${hq}"/>
-        <xacro:wheel prefix="${prefix}right_" parent="${prefix}flipper_link" y_origin="-${y_origin}" reflect="false" hq="${hq}"/>
+        <xacro:wheel prefix="${prefix}left_" parent="${prefix}flipper_link" y_origin="${y_origin}" reflect="false"/>
+        <xacro:wheel prefix="${prefix}right_" parent="${prefix}flipper_link" y_origin="-${y_origin}" reflect="false"/>
         <xacro:flipper_transmission prefix="${prefix}"/>
         <xacro:front_flipper_gazebo prefix="${prefix}"/>

Commit message: rising_description: flippers from continuous to revolute

File: rising_description/urdf/flippers/back_flipper.urdf.xacro (robot description, xacro)
@@ -15,11 +15,10 @@
 	<xacro:property name="y_origin" value="0.274"/>
     <xacro:macro name="back_flipper" params="prefix parent *origin">
-        <joint name="${prefix}flipper_joint" type="continuous">
+        <joint name="${prefix}flipper_joint" type="revolute">
             <parent link="${parent}"/>
             <child link="${prefix}flipper_link"/>
             <xacro:insert_block name="origin"/>
             <axis xyz="0 1 0" rpy="0 0 0"/>
-            <limit effort="100" velocity="10"/>
-            <joint_properties damping="0.5" friction="0.5"/>
+            <limit lower="-3" upper="3" velocity="1.0" effort="10"/>
         </joint>
         <link name="${prefix}flipper_link">

File: rising_description/urdf/flippers/front_flipper.urdf.xacro (robot description, xacro)
@@ -15,11 +15,10 @@
 	<xacro:property name="y_origin" value="0.278"/>
     <xacro:macro name="front_flipper" params="prefix parent *origin">
-        <joint name="${prefix}flipper_joint" type="continuous">
+        <joint name="${prefix}flipper_joint" type="revolute">
             <parent link="${parent}"/>
             <child link="${prefix}flipper_link"/>
             <xacro:insert_block name="origin"/>
             <axis xyz="0 1 0" rpy="0 0 0"/>
-            <limit effort="100" velocity="10"/>
-            <joint_properties damping="0.5" friction="0.5"/>
+            <limit lower="-3" upper="3" velocity="1.0" effort="10"/>
         </joint>
         <link name="${prefix}flipper_link">
