Commit message: Changed color to black

File: rising_description/urdf/base/rising_base.urdf.xacro (robot description, xacro)
@@ -59,4 +59,5 @@
             </collision>
         </link>
+       <xacro:gazebo_colors prefix="${prefix}"/>
     </xacro:macro>
 </robot>

File: rising_description/urdf/common.gazebo.xacro (robot description, xacro)
@@ -17,5 +17,7 @@
 		</gazebo>
 		<gazebo reference="$(arg prefix)base_link">
-			<material>Gazebo/Grey</material>
+			<!--material>Gazebo/Grey</material-->
+			<uri>file://media/materials/scripts/gazebo.material</uri>
+		    <material>Gazebo/Black</material>
 		</gazebo>
 	</xacro:macro>

Commit message: Redefine color gazebo paramenters

File: rising_description/urdf/base/rising_base.urdf.xacro (robot description, xacro)
@@ -33,5 +33,4 @@
                 <mass value="${base_mass}"/>
                 <origin xyz="0 0 0.11"/>
-                <!-- DUDA: Valores -->
                 <solid_cuboid_inertia w="${lenght_on_x}" h="${lenght_on_y}" d="${lenght_on_z}" m="${base_mass}"/>
             </inertial>

File: rising_description/urdf/common.gazebo.xacro (robot description, xacro)
@@ -13,10 +13,5 @@
    </xacro:macro>
    <xacro:macro name="gazebo_colors" params="prefix">
-		<gazebo reference="$(arg prefix)base_footprint">
-			<material>Gazebo/Green</material>
-		</gazebo>
 		<gazebo reference="$(arg prefix)base_link">
-			<!--material>Gazebo/Grey</material-->
-			<uri>file://media/materials/scripts/gazebo.material</uri>
 		    <material>Gazebo/Black</material>
 		</gazebo>

Commit message: rising_description: update base link z position

File: rising_description/urdf/base/rising_base.urdf.xacro (robot description, xacro)
@@ -10,26 +10,16 @@
         <xacro:property name="lenght_on_y" value="0.45"/>
         <xacro:property name="lenght_on_z" value="0.36"/>
-        <!-- BASE FOOTPRINT -->
-        <xacro:if value="${publish_bf}">
-            <link name="${prefix}base_footprint">
-                <visual>
-                    <origin xyz="0 0 0" rpy="0 0 0"/>
-                    <geometry>
-                        <box size="0.001 0.001 0.001"/>
-                    </geometry>
-                </visual>
-            </link>
-            <joint name="${prefix}base_footprint_joint" type="fixed">
-                <!-- DUDA: Valores -->
-                <origin xyz="0 0 0" rpy="0 0 0"/>
-                <parent link="${prefix}base_footprint"/>
-                <child link="${prefix}base_link"/>
-            </joint>
-        </xacro:if>
-        <!-- BASE_LINK -->
+        <!-- Base footprint -->
+        <link name="${prefix}base_footprint"/>
+        <joint name="${prefix}base_footprint_joint" type="fixed">
+            <origin xyz="0 0 0.15407" rpy="0 0 0"/>
+            <parent link="${prefix}base_footprint"/>
+            <child link="${prefix}base_link"/>
+        </joint>
+        <!-- Base link -->
         <link name="${prefix}base_link">
             <inertial>
                 <mass value="${base_mass}"/>
-                <origin xyz="0 0 0.11"/>
+                <origin xyz="0 0 0"/>
                 <solid_cuboid_inertia w="${lenght_on_x}" h="${lenght_on_y}" d="${lenght_on_z}" m="${base_mass}"/>
             </inertial>
@@ -53,5 +43,5 @@
                 <origin xyz="0 0 0" rpy="0 0 0 "/>
 		        <geometry>
-			        <mesh filename="package://rising_description/meshes/base/rising_base_final.stl"/>
+			        <mesh filename="package://rising_description/meshes/base/rising_base_final.dae"/>
                 </geometry>
             </collision>

Commit message: rising_description: update rising base mesh

File: rising_description/urdf/base/rising_base.urdf.xacro (robot description, xacro)
@@ -2,5 +2,5 @@
 <robot name="base" xmlns:xacro="http://www.ros.org/wiki/xacro">
 <xacro:include filename="$(find rising_description)/urdf/inertia.urdf.xacro" />
-    <xacro:macro name="rising_base" params="prefix publish_bf hq">
+    <xacro:macro name="rising_base" params="prefix">
     <!--<xacro:property name="flippers_width" value="0.1"/> -->
         <!-- Robot mechanical and motor parameters -->
@@ -26,14 +26,7 @@
             <visual>
                 <origin xyz="0 0 0" rpy="0 0 0"/>
-                <xacro:if value="${hq}">
-                    <geometry>
-                        <mesh filename="package://rising_description/meshes/base/rising_base_final.dae"/>
-                    </geometry>
-                </xacro:if>
-                <xacro:unless value="${hq}">
-                    <geometry>
-                        <mesh filename="package://rising_description/meshes/base/rising_base_final.stl"/>
-                    </geometry>
-                </xacro:unless>
+                <geometry>
+                    <mesh filename="package://rising_description/meshes/base/rising_base_final.dae"/>
+                </geometry>
                 <material name="dark_grey">
 			        <color rgba="0.4 0.4 0.4 1.0"/>

Commit message: add new cover to urdf

File: rising_description/urdf/base/rising_base.urdf.xacro (robot description, xacro)
@@ -25,4 +25,9 @@
                 <parent link="${prefix}base_footprint"/>
                 <child link="${prefix}base_link"/>
+            </joint>
+            <joint name="${prefix}cover_joint" type="fixed">
+                <origin xyz="0 0 0" rpy="0 0 0"/>
+                <parent link="${prefix}base_footprint"/>
+                <child link="${prefix}cover_link"/>
             </joint>
         </xacro:if>
@@ -57,4 +62,34 @@
             </collision>
         </link>
+        <!-- COVER LINK -->
+        <link name="${prefix}cover_link">
+            <inertial>
+                <mass value="1"/>
+                <origin xyz="0 0 0.29"/>
+                <solid_cuboid_inertia w="${lenght_on_x}" h="${lenght_on_y}" d="0.10" m="1"/>
+            </inertial>
+            <visual>
+                <origin xyz="0 0 0.29" rpy="${PI/2} 0 ${PI/2}"/>
+                <xacro:if value="${hq}">
+                    <geometry>
+                        <mesh filename="package://rising_description/meshes/base/rising_joroba.stl"/>
+                    </geometry>
+                </xacro:if>
+                <xacro:unless value="${hq}">
+                    <geometry>
+                        <mesh filename="package://rising_description/meshes/base/rising_joroba.stl"/>
+                    </geometry>
+                </xacro:unless>
+                <material name="dark_grey">
+			        <color rgba="0.4 0.4 0.4 1.0"/>
+                </material>
+            </visual>
+            <collision>
+                <origin xyz="0 0 0.29" rpy="${PI/2} 0 ${PI/2}"/>
+		        <geometry>
+			        <mesh filename="package://rising_description/meshes/base/rising_joroba.stl"/>
+                </geometry>
+            </collision>
+        </link>
        <xacro:gazebo_colors prefix="${prefix}"/>
     </xacro:macro>
