Commit message: Updated version with arm and gripper

File: rising_description/robots/rising_std.urdf.xacro (robot description, xacro)
@@ -11,6 +11,11 @@
 	<xacro:include filename="$(find rising_description)/urdf/flippers/back_flipper.urdf.xacro" />
     <xacro:include filename="$(find rising_description)/urdf/flippers/front_flipper.urdf.xacro" />
-	<!-- Import all available sensors
-	<xacro:include filename="$(find robotnik_sensors)/urdf/all_sensors.urdf.xacro" />-->
+	<!--Import all available sensors -->
+	<xacro:include filename="$(find robotnik_sensors)/urdf/all_sensors.urdf.xacro" />
+	 <!-- Include KINOVA GEN3 ARM -->
+	<xacro:include filename="$(find kortex_description)/arms/gen3/6dof/urdf/gen3_macro.xacro" />
+	<xacro:include filename="$(find kortex_description)/arms/gen3/6dof/urdf/gen3_transmission_macro.xacro" />
+	<!-- Include KINOVA GEN3 GRIPPER -->
+	<xacro:include filename="$(find kortex_description)/grippers/gen3_lite_2f/urdf/gen3_lite_2f_macro.xacro" />
 	<xacro:property name="PI" value="3.1415926535897931"/>
 	<!-- Flipper parameters -->
@@ -22,5 +27,19 @@
     <xacro:property name="publish_bf" value="true"/>
     <xacro:arg name="prefix" default="rising_"/>
-    <xacro:macro name="rising" params="prefix publish_bf hq">
+	<xacro:arg name="has_arm" default="true"/>
+	<xacro:arg name="has_gripper" default="true"/>
+    <xacro:property name="arm_position_x" value="0.0"/>
+    <xacro:property name="arm_position_y" value="0"/>
+    <xacro:property name="arm_position_z" value="0.1835"/>
+    <xacro:property name="arm_orientation_r" value="0"/>
+    <xacro:property name="arm_orientation_p" value="0"/>
+    <xacro:property name="arm_orientation_y" value="0"/>
+	<xacro:property name="gripper_position_x" value="0.0"/>
+    <xacro:property name="gripper_position_y" value="0"/>
+    <xacro:property name="gripper_position_z" value="0.3135"/>
+    <xacro:property name="gripper_orientation_r" value="0"/>
+    <xacro:property name="gripper_orientation_p" value="0"/>
+    <xacro:property name="gripper_orientation_y" value="0"/>
+    <xacro:macro name="rising" params="prefix publish_bf hq has_arm has_gripper">
 		<!-- *************** -->
 		<!-- Robots Elements -->
@@ -35,4 +54,21 @@
   			<origin xyz="-${flipper_offset_x} -${flipper_offset_y} ${flipper_offset_z}" rpy="0 0 0"/>
   		</xacro:back_flipper>
+ <!-- KINOVA GEN3 ARM -->
+        <xacro:if value="$(arg has_arm)">
+	        <xacro:load_arm prefix="$(arg prefix)arm_" dof="6" vision="180" parent="jiji">
+                <origin xyz="0 0 0" rpy="0 0 0"/>
+            </xacro:load_arm>
+            <joint name="$(arg prefix)arm_base_joint" type="fixed">
+                <origin xyz="${arm_position_x} ${arm_position_y} ${arm_position_z}" rpy="${arm_orientation_r} ${arm_orientation_p} ${arm_orientation_y}"/>
+                <parent link="$(arg prefix)base_link" />
+                <child link="$(arg prefix)arm_base_link"/>
+            </joint>
+	        <xacro:load_gazebo_arm_transmissions prefix="$(arg prefix)arm_"/>
+        </xacro:if>
+<!-- KINOVA GEN3 GRIPPER -->
+        <xacro:if value="$(arg has_gripper)">
+            <xacro:load_gripper prefix="$(arg prefix)" parent="$(arg prefix)arm_end_effector_link">
+            </xacro:load_gripper>
+		</xacro:if>
    </xacro:macro>
    <!-- Gazebo ros control pluggins -->
@@ -52,4 +88,4 @@
         <xacro:ros_control/-->
         <!--xacro:gazebo_colors prefix="$(arg prefix)"/-->
-   <xacro:rising prefix="$(arg prefix)" publish_bf="true" hq="true"/>
+   <xacro:rising prefix="$(arg prefix)" publish_bf="true" hq="true"  has_arm="true" has_gripper="true"/>
 </robot>

File: rising_description/urdf/flippers/back_flipper.gazebo.xacro (robot description, xacro)
@@ -3,6 +3,6 @@
     <xacro:macro name="back_flipper_gazebo" params="prefix">
         <gazebo reference="${prefix}flipper_link">
-            <mu1 value="0.0"/>
-			<mu2 value="1.0"/>
+            <mu1 value="1.0"/>
+			<mu2 value="1.00"/>
 			<kp value="10000000.0" />
 			<kd value="1.0" />

File: rising_description/urdf/flippers/back_flipper.urdf.xacro (robot description, xacro)
@@ -21,5 +21,5 @@
             <xacro:insert_block name="origin"/>
             <axis xyz="0 1 0" rpy="0 0 0"/>
-            <limit effort="100" velocity="100"/>
+            <limit effort="100" velocity="10"/>
             <joint_properties damping="0.5" friction="0.5"/>
         </joint>
@@ -40,11 +40,24 @@
                 </xacro:unless>
             </visual>
-            <!--collision>
-              <origin xyz="0 0 0" rpy="0 0 0"/>
+            <collision>
+                  <xacro:if value="${hq}">
+                    <origin xyz="0 0 0" rpy="0 0 0"/>
+                    <geometry>
+                        <mesh filename="package://rising_description/meshes/flippers/collision_back_flippers.dae" scale="0.001 0.001 0.001"/>
+                    </geometry>
+                </xacro:if>
+                <xacro:unless value="${hq}">
+                    <origin xyz="0 0 0" rpy="0 0 0"/>
+                    <!-- change geometry if hq!=true -->
+                    <geometry>
+                        <cylinder length="${back_flipper_height}" radius="${back_flipper_radius}"/>
+                    </geometry>
+                </xacro:unless>
+              <!--origin xyz="0 0 0" rpy="0 0 0"/>
                <geometry>
-                   <mesh filename="package://rising_description/meshes/flippers/back_flippers.dae" />
-                   <!- - <cylinder length="${back_flipper_height}" radius="${back_flipper_radius}" />- ->
-               </geometry>
-            </collision-->
+                   <mesh filename="package://rising_description/meshes/flippers/collision_back_flippers.dae" />
+                   <!- - <cylinder length="${back_flipper_height}" radius="${back_flipper_radius}" /> - ->
+               </geometry-->
+            </collision>
             <inertial>
                 <mass value="${back_flipper_mass}"/>

File: rising_description/urdf/flippers/front_flipper.gazebo.xacro (robot description, xacro)
@@ -3,5 +3,5 @@
     <xacro:macro name="front_flipper_gazebo" params="prefix">
         <gazebo reference="${prefix}flipper_link">
-            <mu1 value="0.0"/>
+            <mu1 value="1.0"/>
 			<mu2 value="1.0"/>
 			<kp value="10000000.0" />

File: rising_description/urdf/flippers/front_flipper.urdf.xacro (robot description, xacro)
@@ -21,5 +21,5 @@
             <xacro:insert_block name="origin"/>
             <axis xyz="0 1 0" rpy="0 0 0"/>
-            <limit effort="100" velocity="100"/>
+            <limit effort="100" velocity="10"/>
             <joint_properties damping="0.5" friction="0.5"/>
         </joint>
@@ -40,11 +40,24 @@
                 </xacro:unless>
             </visual>
-            <!--collision>
-                <origin xyz="0 0 0" rpy="0 0 0"/>
+            <collision>
+              <xacro:if value="${hq}">
+                    <origin xyz="0 0 0" rpy="0 0 0"/>
+                    <geometry>
+                        <mesh filename="package://rising_description/meshes/flippers/collision_front_flippers.dae" scale="0.001 0.001 0.001"/>
+                    </geometry>
+                </xacro:if>
+                <xacro:unless value="${hq}">
+                    <origin xyz="0 0 0" rpy="0 0 0"/>
+                    <!-- change geometry if hq!=true -->
+                    <geometry>
+                        <cylinder length="${front_flipper_height}" radius="${front_flipper_radius}"/>
+                    </geometry>
+                </xacro:unless>
+                <!-- origin xyz="0 0 0" rpy="0 0 0"/>
                 <geometry>
-                   <mesh filename="package://rising_description/meshes/flippers/front_flippers.dae" />
+                   <mesh filename="package://rising_description/meshes/flippers/collision_front_flippers.dae" />
                     <!- - <cylinder length="${front_flipper_height}" radius="${front_flipper_radius}" />- ->
-                </geometry>
-            </collision-->
+                </geometry-->
+            </collision>
             <inertial>
                 <mass value="${front_flipper_mass}"/>

File: rising_description/urdf/wheels/wheel.gazebo.xacro (robot description, xacro)
@@ -3,9 +3,9 @@
     <xacro:macro name="wheel_gazebo" params="prefix">
         <gazebo reference="${prefix}_wheel_link">
-            <mu1 value="1.0"/>
-			<mu2 value="0.5"/>
-			<kp value="10000000.0" />
-			<kd value="1.0" />
-			<fdir1 value="1 0 0"/>
+            <mu1 value="10000"/>
+			      <mu2 value="10000"/>
+			      <kp value="10000000.0" />
+			      <kd value="1.0" />
+		      	<fdir1 value="1 0 0"/>
 			<material>Gazebo/Yellow</material>
             <turnGravityOff>false</turnGravityOff>

Commit message: Updated version with rs_bpearl configuration

File: rising_description/robots/rising_std.urdf.xacro (robot description, xacro)
@@ -18,4 +18,5 @@
 	<!-- Include KINOVA GEN3 GRIPPER -->
 	<xacro:include filename="$(find kortex_description)/grippers/gen3_lite_2f/urdf/gen3_lite_2f_macro.xacro" />
+	<xacro:include filename="$(find kortex_description)/grippers/gen3_lite_2f/urdf/gen3_lite_2f_transmission_macro.xacro" />
 	<xacro:property name="PI" value="3.1415926535897931"/>
 	<!-- Flipper parameters -->
@@ -70,5 +71,16 @@
             <xacro:load_gripper prefix="$(arg prefix)" parent="$(arg prefix)arm_end_effector_link">
             </xacro:load_gripper>
+        <xacro:load_gazebo_gripper_transmissions prefix="$(arg prefix)"/>
 		</xacro:if>
+<!-- LIDAR -->
+        <sensor_rs_bpearl_lidar prefix="${prefix}" parent="${prefix}base_link" prefix_topic="lidar" range_min="1" range_max="15.0" hfov="360.0" hres="0.1" vfov="90.0" vres="2.0" fps="1.0" gpu="true" >
+           <origin xyz="0.27894 0 0.20667" rpy="0 ${M_PI/4} 0"/>
+        </sensor_rs_bpearl_lidar>
+        <!--xacro:sensor_rplidar prefix="${prefix}rplidar" parent="${prefix}base_link" prefix_topic="front_laser" min_angle="3.14159" max_angle="-3.14159"  gpu="true">
+           <origin xyz="0.27894 0 0.20667" rpy="0 ${M_PI/4} 0"/>
+        </xacro:sensor_rplidar-->
+		<!--xacro:sensor_rs_bpearl_lidar2 prefix="${prefix}lidar" parent="${prefix}base_link" prefix_topic="lidar" gpu="false">
+           <origin xyz="0.27894 0 0.20667" rpy="0 ${M_PI/4} 0"/>
+        </xacro:sensor_rs_bpearl_lidar2-->
    </xacro:macro>
    <!-- Gazebo ros control pluggins -->

Commit message: Xacro name changed

File: rising_description/robots/rising_std.urdf.xacro (robot description, xacro)
@@ -74,13 +74,7 @@
 		</xacro:if>
 <!-- LIDAR -->
-        <xacro:sensor_rs_bpearl_lidar prefix="${prefix}" parent="${prefix}base_link" prefix_topic="lidar" range_min="0.1" range_max="90" hfov="360" samples="1200" vfov="90.0" lasers="32" fps="15" gpu="true" >
+        <xacro:sensor_rs_bpearl prefix="${prefix}" parent="${prefix}base_link" prefix_topic="lidar" range_min="0.1" range_max="90" hfov="360" samples="1200" vfov="90.0" lasers="32" fps="15" gpu="true" >
            <origin xyz="0.27894 0 0.20667" rpy="0 ${M_PI/4} 0"/>
-        </xacro:sensor_rs_bpearl_lidar>
-        <!--xacro:sensor_rplidar prefix="${prefix}rplidar" parent="${prefix}base_link" prefix_topic="front_laser" min_angle="3.14159" max_angle="-3.14159"  gpu="true">
-           <origin xyz="0.27894 0 0.20667" rpy="0 ${M_PI/4} 0"/>
-        </xacro:sensor_rplidar-->
-		<!--xacro:sensor_rslidar_16 prefix="${prefix}lidar" parent="${prefix}base_link" prefix_topic="lidar" gpu="false">
-           <origin xyz="0.27894 0 0.20667" rpy="0 ${M_PI/4} 0"/>
-        </xacro:sensor_rslidar_16-->
+        </xacro:sensor_rs_bpearl>
    </xacro:macro>
    <!-- Gazebo ros control pluggins -->

Commit message: Unneeded comments deleted and ARM paramater parent changed

File: rising_description/robots/rising_std.urdf.xacro (robot description, xacro)
@@ -5,6 +5,4 @@
 	<!-- ***************** -->
 	<!-- First we import all posible elements defined in the urdf.xacro files. All these elements are defined as macro:xacros -->
-	<!-- Import rising_platform -->
-    <!--xacro:include filename="$(find rising_description)/robots/rising_platform.urdf.xacro"/-->
 	<!-- Import flippers -->
 	<xacro:include filename="$(find rising_description)/urdf/base/rising_base.urdf.xacro" />
@@ -57,5 +55,5 @@
  <!-- KINOVA GEN3 ARM -->
         <xacro:if value="$(arg has_arm)">
-	        <xacro:load_arm prefix="$(arg prefix)arm_" dof="6" vision="180" parent="jiji">
+	        <xacro:load_arm prefix="$(arg prefix)arm_" dof="6" vision="180" parent="base_link">
                 <origin xyz="0 0 0" rpy="0 0 0"/>
             </xacro:load_arm>

File: rising_description/urdf/wheels/wheel.transmission.xacro (robot description, xacro)
@@ -14,14 +14,4 @@
             </actuator>
         </transmission>
-        <!--transmission name="${prefix}slave_wheel_joint_trans" params="prefix">
-            <type>transmission_interface/SimpleTransmission</type>
-            <joint name="${prefix}slave_wheel_joint">
-                <hardwareInterface>hardware_interface/VelocityJointInterface</hardwareInterface>
-            </joint>
-            <actuator name="${prefix}slave_wheel_joint_motor">
-				<mechanicalReduction>1</mechanicalReduction>
-				<motorTorqueConstant>20</motorTorqueConstant>
-            </actuator>
-        </transmission-->
     </xacro:macro>
 </robot>

Commit message: Connected arm and gripper launch control parameters

File: rising_description/robots/rising_std.urdf.xacro (robot description, xacro)
@@ -26,5 +26,5 @@
     <xacro:property name="publish_bf" value="true"/>
     <xacro:arg name="prefix" default="rising_"/>
-	<xacro:arg name="has_arm" default="true"/>
+	<xacro:arg name="has_arm" default="false"/>
 	<xacro:arg name="has_gripper" default="true"/>
     <xacro:property name="arm_position_x" value="0.0"/>
@@ -54,20 +54,20 @@
   		</xacro:back_flipper>
  <!-- KINOVA GEN3 ARM -->
-        <xacro:if value="$(arg has_arm)">
-	        <xacro:load_arm prefix="$(arg prefix)arm_" dof="6" vision="180" parent="base_link">
+        <xacro:if value="${has_arm}">
+	        <xacro:load_arm prefix="${prefix}arm_" dof="6" vision="180" parent="${prefix}base_link">
                 <origin xyz="0 0 0" rpy="0 0 0"/>
             </xacro:load_arm>
-            <joint name="$(arg prefix)arm_base_joint" type="fixed">
+            <joint name="${prefix}arm_base_joint" type="fixed">
                 <origin xyz="${arm_position_x} ${arm_position_y} ${arm_position_z}" rpy="${arm_orientation_r} ${arm_orientation_p} ${arm_orientation_y}"/>
-                <parent link="$(arg prefix)base_link" />
-                <child link="$(arg prefix)arm_base_link"/>
+                <parent link="${prefix}base_link" />
+                <child link="${prefix}arm_base_link"/>
             </joint>
-	        <xacro:load_gazebo_arm_transmissions prefix="$(arg prefix)arm_"/>
+	        <xacro:load_gazebo_arm_transmissions prefix="${prefix}arm_"/>
         </xacro:if>
 <!-- KINOVA GEN3 GRIPPER -->
-        <xacro:if value="$(arg has_gripper)">
-            <xacro:load_gripper prefix="$(arg prefix)" parent="$(arg prefix)arm_end_effector_link">
+        <xacro:if value="${has_gripper}">
+            <xacro:load_gripper prefix="${prefix}" parent="${prefix}arm_end_effector_link">
             </xacro:load_gripper>
-        <xacro:load_gazebo_gripper_transmissions prefix="$(arg prefix)"/>
+        <xacro:load_gazebo_gripper_transmissions prefix="${prefix}"/>
 		</xacro:if>
 <!-- LIDAR -->
@@ -92,4 +92,4 @@
         <xacro:ros_control/-->
         <!--xacro:gazebo_colors prefix="$(arg prefix)"/-->
-   <xacro:rising prefix="$(arg prefix)" publish_bf="true" hq="true"  has_arm="true" has_gripper="true"/>
+   <xacro:rising prefix="$(arg prefix)" publish_bf="true" hq="true"  has_arm="$(arg has_arm)" has_gripper="$(arg has_gripper)"/>
 </robot>

Commit message: Updated rising model

File: rising_description/robots/rising_std.urdf.xacro (robot description, xacro)
@@ -5,4 +5,5 @@
 	<!-- ***************** -->
 	<!-- First we import all posible elements defined in the urdf.xacro files. All these elements are defined as macro:xacros -->
+    <xacro:include filename="$(find rising_description)/urdf/common.gazebo.xacro" />
 	<!-- Import flippers -->
 	<xacro:include filename="$(find rising_description)/urdf/base/rising_base.urdf.xacro" />
@@ -72,5 +73,5 @@
 		</xacro:if>
 <!-- LIDAR -->
-        <xacro:sensor_rs_bpearl prefix="${prefix}" parent="${prefix}base_link" prefix_topic="lidar" range_min="0.1" range_max="90" hfov="360" samples="1200" vfov="90.0" lasers="32" fps="15" gpu="true" >
+        <xacro:sensor_rs_bpearl prefix="${prefix}" parent="${prefix}base_link" prefix_topic="lidar" range_min="0.1" range_max="90" hfov="360" samples="1200" vfov="90.0" lasers="32" fps="15" gpu="false" >
            <origin xyz="0.27894 0 0.20667" rpy="0 ${M_PI/4} 0"/>
         </xacro:sensor_rs_bpearl>

File: rising_description/urdf/base/rising_base.urdf.xacro (robot description, xacro)
@@ -2,5 +2,4 @@
 <robot name="base" xmlns:xacro="http://www.ros.org/wiki/xacro">
 <xacro:include filename="$(find rising_description)/urdf/inertia.urdf.xacro" />
-<xacro:include filename="$(find rising_description)/urdf/common.gazebo.xacro" />
     <xacro:macro name="rising_base" params="prefix publish_bf hq">
     <!--<xacro:property name="flippers_width" value="0.1"/> -->
@@ -39,10 +38,10 @@
                 <xacro:if value="${hq}">
                     <geometry>
-                        <mesh filename="package://rising_description/meshes/base/rising_base.dae"/>
+                        <mesh filename="package://rising_description/meshes/base/rising_base_final.dae"/>
                     </geometry>
                 </xacro:if>
                 <xacro:unless value="${hq}">
                     <geometry>
-                        <mesh filename="package://rising_description/meshes/base/rising_base.stl"/>
+                        <mesh filename="package://rising_description/meshes/base/rising_base_final.stl"/>
                     </geometry>
                 </xacro:unless>
@@ -54,5 +53,5 @@
                 <origin xyz="0 0 0" rpy="0 0 0 "/>
 		        <geometry>
-			        <mesh filename="package://rising_description/meshes/base/rising_base.stl"/>
+			        <mesh filename="package://rising_description/meshes/base/rising_base_final.stl"/>
                 </geometry>
             </collision>

File: rising_description/urdf/flippers/back_flipper.urdf.xacro (robot description, xacro)
@@ -28,5 +28,5 @@
                     <origin xyz="0 0 0" rpy="0 0 0"/>
                     <geometry>
-                        <mesh filename="package://rising_description/meshes/flippers/back_flippers.dae"/>
+                        <mesh filename="package://rising_description/meshes/flippers/back_flippers_final.dae"/>
                     </geometry>
                 </xacro:if>
@@ -41,11 +41,11 @@
             <collision>
                   <xacro:if value="${hq}">
-                    <origin xyz="0 0 0" rpy="0 0 0"/>
+                    <origin xyz="-0.13688 0 0" rpy="${M_PI/2} 0 0"/>
                     <geometry>
-                        <mesh filename="package://rising_description/meshes/flippers/collision_back_flippers.dae" scale="0.001 0.001 0.001"/>
+                        <mesh filename="package://rising_description/meshes/flippers/collision_back_flippers_final.dae" scale="0.001 0.001 0.001"/>
                     </geometry>
                 </xacro:if>
                 <xacro:unless value="${hq}">
-                    <origin xyz="0 0 0" rpy="0 0 0"/>
+                    <origin xyz="-0.13688 0 0" rpy="${M_PI/2} 0 0"/>
                     <!-- change geometry if hq!=true -->
                     <geometry>

File: rising_description/urdf/flippers/front_flipper.urdf.xacro (robot description, xacro)
@@ -28,5 +28,5 @@
                     <origin xyz="0 0 0" rpy="0 0 0"/>
                     <geometry>
-                        <mesh filename="package://rising_description/meshes/flippers/front_flippers.dae"/>
+                        <mesh filename="package://rising_description/meshes/flippers/front_flippers_final.dae"/>
                     </geometry>
                 </xacro:if>
@@ -43,5 +43,5 @@
                     <origin xyz="0 0 0" rpy="0 0 0"/>
                     <geometry>
-                        <mesh filename="package://rising_description/meshes/flippers/collision_front_flippers.dae" scale="0.001 0.001 0.001"/>
+                        <mesh filename="package://rising_description/meshes/flippers/collision_front_flippers_final.dae" scale="0.001 0.001 0.001"/>
                     </geometry>
                 </xacro:if>
