Commit message: rising_description: update robot definition

File: rising_description/robots/rising_std.urdf.xacro (robot description, xacro)
@@ -12,7 +12,7 @@
 	<!--Import all available sensors -->
 	<xacro:include filename="$(find robotnik_sensors)/urdf/all_sensors.urdf.xacro" />
-	 <!-- Include KINOVA GEN3 ARM -->
-	<xacro:include filename="$(find kortex_description)/arms/gen3/6dof/urdf/gen3_macro.xacro" />
-	<xacro:include filename="$(find kortex_description)/arms/gen3/6dof/urdf/gen3_transmission_macro.xacro" />
+	<!-- Import kinova arm -->
+	<xacro:include filename="$(find rising_description)/urdf/arm/kinova/gen3_macro.xacro" />
+	<xacro:include filename="$(find rising_description)/urdf/arm/kinova/gen3_transmission_macro.xacro" />
 	<!-- Include KINOVA GEN3 GRIPPER -->
 	<xacro:include filename="$(find kortex_description)/grippers/gen3_lite_2f/urdf/gen3_lite_2f_macro.xacro" />
@@ -20,7 +20,7 @@
 	<xacro:property name="PI" value="3.1415926535897931"/>
 	<!-- Flipper parameters -->
-	<xacro:property name="flipper_offset_x" value="0.27455" />    <!-- x,y,z in translation from base_link to the center of the flippers -->
+	<xacro:property name="flipper_offset_x" value="0.325" />    <!-- x,y,z in translation from base_link to the center of the flippers -->
     <xacro:property name="flipper_offset_y" value="0.0" />
-	<xacro:property name="flipper_offset_z" value="0.00" />
+	<xacro:property name="flipper_offset_z" value="0.0" />
 	<!-- Flag to select the high or low quality model -->
 	<xacro:property name="hq" value="true" />
@@ -48,11 +48,13 @@
 		<!-- Rising base -->
 		<xacro:rising_base prefix="$(arg prefix)" publish_bf="${publish_bf}" hq="${hq}" />
-  		<xacro:front_flipper prefix="$(arg prefix)front_" parent="$(arg prefix)base_link" hq="${hq}">
-  			<origin xyz="${flipper_offset_x} -${flipper_offset_y} ${flipper_offset_z}" rpy="0 0 0"/>
+        <!-- Flippers -->
+  		<xacro:front_flipper prefix="$(arg prefix)front_" parent="$(arg prefix)base_link">
+  			<origin xyz="${flipper_offset_x} ${flipper_offset_y} ${flipper_offset_z}" rpy="0 0 0"/>
+  			<!--origin xyz="1 1 1" rpy="0 0 0"/-->
   		</xacro:front_flipper>
-  		<xacro:back_flipper prefix="$(arg prefix)back_" parent="$(arg prefix)base_link" hq="${hq}">
-  			<origin xyz="-${flipper_offset_x} -${flipper_offset_y} ${flipper_offset_z}" rpy="0 0 0"/>
+  		<xacro:back_flipper prefix="$(arg prefix)back_" parent="$(arg prefix)base_link">
+  			<origin xyz="-${flipper_offset_x} ${flipper_offset_y} ${flipper_offset_z}" rpy="0 0 0"/>
   		</xacro:back_flipper>
- <!-- KINOVA GEN3 ARM -->
+        <!-- Arm -->
         <xacro:if value="${has_arm}">
 	        <xacro:load_arm prefix="${prefix}arm_" dof="6" vision="180" parent="${prefix}base_link">
@@ -64,33 +66,19 @@
                 <child link="${prefix}arm_base_link"/>
             </joint>
-	        <xacro:load_gazebo_arm_transmissions prefix="${prefix}arm_"/>
+            <xacro:load_gazebo_arm_transmissions prefix="${prefix}arm_"/>
         </xacro:if>
-<!-- KINOVA GEN3 GRIPPER -->
-        <xacro:if value="${has_gripper}">
+        <!-- Gripper -->
+        <!--xacro:if value="${has_gripper}">
             <xacro:load_gripper prefix="${prefix}" parent="${prefix}arm_end_effector_link">
             </xacro:load_gripper>
-        <xacro:load_gazebo_gripper_transmissions prefix="${prefix}"/>
-		</xacro:if>
-<!-- LIDAR -->
-        <xacro:sensor_rs_bpearl prefix="${prefix}" parent="${prefix}base_link" prefix_topic="lidar" range_min="0.1" range_max="90" hfov="360" samples="1200" vfov="90.0" lasers="32" fps="15" gpu="false" >
-           <origin xyz="0.27894 0 0.20667" rpy="0 ${M_PI/4} 0"/>
+            <xacro:load_gazebo_gripper_transmissions prefix="${prefix}"/>
+	    </xacro:if-->
+        <!-- Sensors -->
+        <xacro:sensor_rs_bpearl prefix="${prefix}rsbpearl" parent="${prefix}base_link" prefix_topic="lidar" range_min="0.1" range_max="90" hfov="360" samples="1200" vfov="90.0" lasers="32" fps="15" gpu="false" >
+            <origin xyz="0.27894 0 0.20667" rpy="0 ${M_PI/4} 0"/>
         </xacro:sensor_rs_bpearl>
-   </xacro:macro>
+    </xacro:macro>
    <!-- Gazebo ros control pluggins -->
    <xacro:ros_control/>
-	<!--xacro:if value="$(arg ros_planar_move_plugin)">
-		<xacro:if value="$(arg omni_wheels)">
-			<xacro:omni_steering prefix="$(arg prefix)" publish_tf="true"/>
-		</xacro:if>
-		<xacro:unless value="$(arg omni_wheels)">
-			<xacro:skid_steering prefix="$(arg prefix)" publish_tf="true"/>
-		</xacro:unless>
-	</xacro:if> -->
-	        <!-- ************** -->
-        <!-- GAZEBO PLUGINS -->
-        <!-- ************** -->
-        <!-- Gazebo ros control pluggins >
-        <xacro:ros_control/-->
-        <!--xacro:gazebo_colors prefix="$(arg prefix)"/-->
    <xacro:rising prefix="$(arg prefix)" publish_bf="true" hq="true"  has_arm="$(arg has_arm)" has_gripper="$(arg has_gripper)"/>
 </robot>

Commit message: update rising common

File: rising_description/robots/rising_std.urdf.xacro (robot description, xacro)
@@ -13,9 +13,9 @@
 	<xacro:include filename="$(find robotnik_sensors)/urdf/all_sensors.urdf.xacro" />
 	 <!-- Include KINOVA GEN3 ARM -->
-	<xacro:include filename="$(find kortex_description)/arms/gen3/6dof/urdf/gen3_macro.xacro" />
-	<xacro:include filename="$(find kortex_description)/arms/gen3/6dof/urdf/gen3_transmission_macro.xacro" />
+	<!--xacro:include filename="$(find kortex_description)/arms/gen3/6dof/urdf/gen3_macro.xacro" />
+	<xacro:include filename="$(find kortex_description)/arms/gen3/6dof/urdf/gen3_transmission_macro.xacro" /-->
 	<!-- Include KINOVA GEN3 GRIPPER -->
-	<xacro:include filename="$(find kortex_description)/grippers/gen3_lite_2f/urdf/gen3_lite_2f_macro.xacro" />
-	<xacro:include filename="$(find kortex_description)/grippers/gen3_lite_2f/urdf/gen3_lite_2f_transmission_macro.xacro" />
+	<!--xacro:include filename="$(find kortex_description)/grippers/gen3_lite_2f/urdf/gen3_lite_2f_macro.xacro" />
+	<xacro:include filename="$(find kortex_description)/grippers/gen3_lite_2f/urdf/gen3_lite_2f_transmission_macro.xacro" /-->
 	<xacro:property name="PI" value="3.1415926535897931"/>
 	<!-- Flipper parameters -->
@@ -28,5 +28,5 @@
     <xacro:arg name="prefix" default="rising_"/>
 	<xacro:arg name="has_arm" default="false"/>
-	<xacro:arg name="has_gripper" default="true"/>
+	<xacro:arg name="has_gripper" default="false"/>
     <xacro:property name="arm_position_x" value="0.0"/>
     <xacro:property name="arm_position_y" value="0"/>
@@ -49,8 +49,8 @@
 		<xacro:rising_base prefix="$(arg prefix)" publish_bf="${publish_bf}" hq="${hq}" />
   		<xacro:front_flipper prefix="$(arg prefix)front_" parent="$(arg prefix)base_link" hq="${hq}">
-  			<origin xyz="${flipper_offset_x} -${flipper_offset_y} ${flipper_offset_z}" rpy="0 0 0"/>
+  			<origin xyz="${flipper_offset_x} -${flipper_offset_y} ${flipper_offset_z}" rpy="0 -1.57 0"/>
   		</xacro:front_flipper>
   		<xacro:back_flipper prefix="$(arg prefix)back_" parent="$(arg prefix)base_link" hq="${hq}">
-  			<origin xyz="-${flipper_offset_x} -${flipper_offset_y} ${flipper_offset_z}" rpy="0 0 0"/>
+  			<origin xyz="-${flipper_offset_x} -${flipper_offset_y} ${flipper_offset_z}" rpy="0 1.57 0"/>
   		</xacro:back_flipper>
  <!-- KINOVA GEN3 ARM -->
@@ -73,7 +73,17 @@
 		</xacro:if>
 <!-- LIDAR -->
-        <xacro:sensor_rs_bpearl prefix="${prefix}" parent="${prefix}base_link" prefix_topic="lidar" range_min="0.1" range_max="90" hfov="360" samples="1200" vfov="90.0" lasers="32" fps="15" gpu="false" >
+        <xacro:sensor_rs_bpearl prefix="${prefix}front_3d_laser" parent="${prefix}base_link" prefix_topic="front_3d_laser" range_min="0.1" range_max="90" hfov="360" samples="1200" vfov="90.0" lasers="32" fps="15" gpu="false" >
            <origin xyz="0.27894 0 0.20667" rpy="0 ${M_PI/4} 0"/>
         </xacro:sensor_rs_bpearl>
+<!-- CAMERAS -->
+        <xacro:sensor_intel_d435 prefix="${prefix}front_rgbd_camera" parent="${prefix}base_link" prefix_topic="front_rgbd_camera" use_nominal_extrinsics="true" >
+           <origin xyz="0.408 0 0.00225" rpy="0 0 0"/>
+        </xacro:sensor_intel_d435>
+        <xacro:sensor_intel_d435 prefix="${prefix}back_rgbd_camera" parent="${prefix}base_link" prefix_topic="back_rgbd_camera" use_nominal_extrinsics="true">
+           <origin xyz="-0.408 0 0.0023" rpy="0 0 3.14"/>
+        </xacro:sensor_intel_d435>
+<xacro:sensor_imu_hector prefix="$(arg prefix)imu" parent="$(arg prefix)base_link">
+		<origin xyz="0.07136 0.0365 0.2711" rpy="0 0 0"/>
+	</xacro:sensor_imu_hector>
    </xacro:macro>
    <!-- Gazebo ros control pluggins -->

File: rising_description/urdf/flippers/back_flipper.urdf.xacro (robot description, xacro)
@@ -20,5 +20,5 @@
             <xacro:insert_block name="origin"/>
             <axis xyz="0 1 0" rpy="0 0 0"/>
-            <limit effort="100" velocity="10"/>
+            <limit effort="100" velocity="100"/>
             <joint_properties damping="0.5" friction="0.5"/>
         </joint>
@@ -28,5 +28,5 @@
                     <origin xyz="0 0 0" rpy="0 0 0"/>
                     <geometry>
-                        <mesh filename="package://rising_description/meshes/flippers/back_flippers_final.dae"/>
+                        <mesh filename="package://rising_description/meshes/flippers/back_flippers.dae"/>
                     </geometry>
                 </xacro:if>

File: rising_description/urdf/flippers/front_flipper.urdf.xacro (robot description, xacro)
@@ -20,5 +20,5 @@
             <xacro:insert_block name="origin"/>
             <axis xyz="0 1 0" rpy="0 0 0"/>
-            <limit effort="100" velocity="10"/>
+            <limit effort="100" velocity="100"/>
             <joint_properties damping="0.5" friction="0.5"/>
         </joint>
@@ -28,5 +28,5 @@
                     <origin xyz="0 0 0" rpy="0 0 0"/>
                     <geometry>
-                        <mesh filename="package://rising_description/meshes/flippers/front_flippers_final.dae"/>
+                        <mesh filename="package://rising_description/meshes/flippers/front_flippers.dae"/>
                     </geometry>
                 </xacro:if>

File: rising_description/urdf/wheels/wheel.urdf.xacro (robot description, xacro)
@@ -22,5 +22,5 @@
             <origin xyz="0 ${y_origin} 0" rpy="0 0 0"/>
             <axis xyz="0 1 0" rpy="0 0 0"/>
-            <limit effort="100" velocity="100"/>
+            <limit effort="100" velocity="600"/>
             <joint_properties damping="0.0" friction="0.0"/>
         </joint>
@@ -54,5 +54,5 @@
             </xacro:unless>
             <axis xyz="0 1 0" rpy="0 0 0"/>
-            <limit effort="100" velocity="100"/>
+            <limit effort="100" velocity="600"/>
             <mimic joint="{prefix}master_wheel_joint" multiplier="${multiplier}" offset="0" />
             <joint_properties damping="0.0" friction="0.0"/>
@@ -87,5 +87,5 @@
             </xacro:unless>
             <axis xyz="0 1 0" rpy="0 0 0"/>
-            <limit effort="100" velocity="100"/>
+            <limit effort="100" velocity="600"/>
             <mimic joint="{prefix}master_wheel_joint" multiplier="${multiplier}" offset="0" />
             <joint_properties damping="0.0" friction="0.0"/>
@@ -120,5 +120,5 @@
             </xacro:unless>
             <axis xyz="0 1 0" rpy="0 0 0"/>
-            <limit effort="100" velocity="100"/>
+            <limit effort="100" velocity="600"/>
             <mimic joint="{prefix}master_wheel_joint" multiplier="${multiplier}" offset="0" />
             <joint_properties damping="0.0" friction="0.0"/>
@@ -153,5 +153,5 @@
             </xacro:unless>
             <axis xyz="0 1 0" rpy="0 0 0"/>
-            <limit effort="100" velocity="100"/>
+            <limit effort="100" velocity="600"/>
             <mimic joint="{prefix}master_wheel_joint" multiplier="${multiplier}" offset="0" />
             <joint_properties damping="0.0" friction="0.0"/>

Commit message: add changes

File: rising_description/robots/rising_std.urdf.xacro (robot description, xacro)
@@ -20,5 +20,5 @@
 	<xacro:property name="PI" value="3.1415926535897931"/>
 	<!-- Flipper parameters -->
-	<xacro:property name="flipper_offset_x" value="0.27455" />    <!-- x,y,z in translation from base_link to the center of the flippers -->
+	<xacro:property name="flipper_offset_x" value="0.31455" />    <!-- x,y,z in translation from base_link to the center of the flippers -->
     <xacro:property name="flipper_offset_y" value="0.0" />
 	<xacro:property name="flipper_offset_z" value="0.00" />
@@ -34,5 +34,5 @@
     <xacro:property name="arm_orientation_r" value="0"/>
     <xacro:property name="arm_orientation_p" value="0"/>
-    <xacro:property name="arm_orientation_y" value="0"/>
+    <xacro:property name="arm_orientation_y" value="${M_PI}"/>
 	<xacro:property name="gripper_position_x" value="0.0"/>
     <xacro:property name="gripper_position_y" value="0"/>
@@ -49,8 +49,8 @@
 		<xacro:rising_base prefix="$(arg prefix)" publish_bf="${publish_bf}" hq="${hq}" />
   		<xacro:front_flipper prefix="$(arg prefix)front_" parent="$(arg prefix)base_link" hq="${hq}">
-  			<origin xyz="${flipper_offset_x} -${flipper_offset_y} ${flipper_offset_z}" rpy="0 -1.57 0"/>
+  			<origin xyz="${flipper_offset_x} -${flipper_offset_y} ${flipper_offset_z}" rpy="0 -3.14 0"/>
   		</xacro:front_flipper>
   		<xacro:back_flipper prefix="$(arg prefix)back_" parent="$(arg prefix)base_link" hq="${hq}">
-  			<origin xyz="-${flipper_offset_x} -${flipper_offset_y} ${flipper_offset_z}" rpy="0 1.57 0"/>
+  			<origin xyz="-${flipper_offset_x} -${flipper_offset_y} ${flipper_offset_z}" rpy="0 3.14 0"/>
   		</xacro:back_flipper>
  <!-- KINOVA GEN3 ARM -->

File: rising_description/urdf/base/rising_base.urdf.xacro (robot description, xacro)
@@ -30,4 +30,9 @@
                 <parent link="${prefix}base_footprint"/>
                 <child link="${prefix}cover_link"/>
+            </joint>
+            <joint name="${prefix}arm_support_struct_joint" type="fixed">
+                <origin xyz="0 0 0" rpy="0 0 0"/>
+                <parent link="${prefix}base_footprint"/>
+                <child link="${prefix}arm_support_struct_link"/>
             </joint>
         </xacro:if>
@@ -70,5 +75,5 @@
             </inertial>
             <visual>
-                <origin xyz="0 0 0.29" rpy="${PI/2} 0 ${PI/2}"/>
+                <origin xyz="0 0 0.29" rpy="${PI/2} 0 ${-PI/2}"/>
                 <xacro:if value="${hq}">
                     <geometry>
@@ -86,7 +91,37 @@
             </visual>
             <collision>
-                <origin xyz="0 0 0.29" rpy="${PI/2} 0 ${PI/2}"/>
+                <origin xyz="0 0 0.29" rpy="${PI/2} 0 ${-PI/2}"/>
 		        <geometry>
 			        <mesh filename="package://rising_description/meshes/base/rising_joroba.stl"/>
+                </geometry>
+            </collision>
+        </link>
+        <!-- ARM SUPPORT STRUCTURE -->
+        <link name="${prefix}arm_support_struct_link">
+            <inertial>
+                <mass value="1"/>
+                <origin xyz="-0.3228 0 0.21315"/>
+                <solid_cuboid_inertia w="0.10" h="0.10" d="0.10" m="1"/>
+            </inertial>
+            <visual>
+                <origin xyz="-0.3228 0 0.21315" rpy="0 0 0"/>
+                <xacro:if value="${hq}">
+                    <geometry>
+                        <mesh filename="package://rising_description/meshes/base/rising_kinova_support.stl"/>
+                    </geometry>
+                </xacro:if>
+                <xacro:unless value="${hq}">
+                    <geometry>
+                        <mesh filename="package://rising_description/meshes/base/rising_kinova_support.stl"/>
+                    </geometry>
+                </xacro:unless>
+                <material name="dark_grey">
+			        <color rgba="0.4 0.4 0.4 1.0"/>
+                </material>
+            </visual>
+            <collision>
+                <origin xyz="-0.3228 0 0.21315" rpy="0 0 0"/>
+		        <geometry>
+			        <mesh filename="package://rising_description/meshes/base/rising_kinova_support.stl"/>
                 </geometry>
             </collision>
